File: Hardware/ControllerPCB/BugWiperPCB.kicad_sch (KiCad schematic)
At the start: 14 parts, among them J2 1770924, J3 Phoenix_1776508, J6 1824420000, J7 Conn_01x02_Pin

Commit message: update BOM
Parts:
- C27: value 100nF -> 100nF; Manufacturer_Name (none) -> Samsung; Manufacturer_Part_Number (none) -> CL10B104KB8NNNC; Mouser Part Number (none) -> 187-CL10B104KB8NNNC; Mouser Price/Stock (none) -> 0,01 €
- F2, F3: Mouser Part Number (none) -> 504-PTS120630V012; Mouser Price/Stock (none) -> 0,108€
- J2: Manufacturer_Name (none) -> Phoenix Contact; Manufacturer_Part_Number (none) -> 1770924; Mouser Part Number (none) -> 651-1770924; Mouser Price/Stock (none) -> 1,29 €
- J3: Manufacturer_Part_Number (none) -> 1776508; Mouser Part Number (none) -> 651-1776508; Mouser Price/Stock (none) -> 1,83 €
- J6: Mouser Price/Stock https://www.mouser.co.uk/ProductDetail/Weidmuller/182442000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 -> 1,11 €
- J7: Manufacturer_Name (none) -> JST; Manufacturer_Part_Number (none) -> B2B-XH-AM(LF)(SN); Mouser Part Number (none) -> 306-B2B-XH-AMLFSNP; Mouser Price/Stock (none) -> 0,152 €
Changed lines of the file:
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@@
+      (effects (font (size 1.27 1.27)) hide)
+    )
+    (property "Mouser Part Number" "504-PTS120630V012" (at 219.71 128.27 0)
+      (effects (font (size 1.27 1.27)) hide)
+    )
+    (property "Mouser Price/Stock" "0,108€" (at 219.71 128.27 0)
       (effects (font (size 1.27 1.27)) hide)
     )
@@
       (effects (font (size 1.27 1.27)) hide)
     )
+    (property "Manufacturer_Name" "Phoenix Contact" (at 242.57 143.51 0)
+      (effects (font (size 1.27 1.27)) hide)
+    )
+    (property "Manufacturer_Part_Number" "1770924" (at 242.57 143.51 0)
+      (effects (font (size 1.27 1.27)) hide)
+    )
+    (property "Mouser Part Number" "651-1770924" (at 242.57 143.51 0)
+      (effects (font (size 1.27 1.27)) hide)
+    )
+    (property "Mouser Price/Stock" "1,29 €" (at 242.57 143.51 0)
+      (effects (font (size 1.27 1.27)) hide)
+    )
     (pin "7")
     (pin "5")
@@
       (effects (font (size 1.27 1.27)) hide)
     )
+    (property "Description" " 2 Pos 5.08mm pitch Through Hole Header" (at 156.21 43.18 0)
+      (effects (font (size 1.27 1.27)) hide)
+    )
+    (property "Manufacturer_Part_Number" "1776508" (at 156.21 43.18 0)
+      (effects (font (size 1.27 1.27)) hide)
+    )
+    (property "Mouser Part Number" "651-1776508" (at 156.21 43.18 0)
+      (effects (font (size 1.27 1.27)) hide)
+    )
+    (property "Mouser Price/Stock" "1,83 €" (at 156.21 43.18 0)
+      (effects (font (size 1.27 1.27)) hide)
+    )
     (pin "1")
     (pin "2")
@@
       (effects (font (size 1.27 1.27)) hide)
     )
+    (property "Mouser Part Number" "504-PTS120630V012" (at 234.95 143.51 0)
+      (effects (font (size 1.27 1.27)) hide)
+    )
+    (property "Mouser Price/Stock" "0,108€" (at 234.95 143.51 0)
+      (effects (font (size 1.27 1.27)) hide)
+    )
     (pin "1")
     (pin "2")
@@
     )
     (property "Alternative Price" "" (at 251.46 102.87 0)
+      (effects (font (size 1.27 1.27)) hide)
+    )
+    (property "Manufacturer_Name" "JST" (at 251.46 102.87 0)
+      (effects (font (size 1.27 1.27)) hide)
+    )
+    (property "Manufacturer_Part_Number" "B2B-XH-AM(LF)(SN)" (at 251.46 102.87 0)
+      (effects (font (size 1.27 1.27)) hide)
+    )
+    (property "Mouser Part Number" "306-B2B-XH-AMLFSNP" (at 251.46 102.87 0)
+      (effects (font (size 1.27 1.27)) hide)
+    )
+    (property "Mouser Price/Stock" "0,152 €" (at 251.46 102.87 0)
       (effects (font (size 1.27 1.27)) hide)
     )
@@
       (effects (font (size 1.27 1.27)) (justify left))
     )
-    (property "Value" "100nF" (at 106.68 172.72 0)
+    (property "Value" "100nF " (at 106.68 172.72 0)
       (effects (font (size 1.27 1.27)) (justify left))
     )
@@
     )
     (property "Alternative Price" "" (at 110.49 171.45 0)
+      (effects (font (size 1.27 1.27)) hide)
+    )
+    (property "Description" "100nF+/-10% 50V X7R 0603" (at 110.49 171.45 0)
+      (effects (font (size 1.27 1.27)) hide)
+    )
+    (property "Manufacturer_Name" "Samsung" (at 110.49 171.45 0)
+      (effects (font (size 1.27 1.27)) hide)
+    )
+    (property "Manufacturer_Part_Number" "CL10B104KB8NNNC" (at 110.49 171.45 0)
+      (effects (font (size 1.27 1.27)) hide)
+    )
+    (property "Mouser Part Number" "187-CL10B104KB8NNNC" (at 110.49 171.45 0)
+      (effects (font (size 1.27 1.27)) hide)
+    )
+    (property "Mouser Price/Stock" "0,01 €" (at 110.49 171.45 0)
       (effects (font (size 1.27 1.27)) hide)
     )
@@
       (effects (font (size 1.27 1.27)) (justify left top) hide)
     )
-    (property "Mouser Price/Stock" "https://www.mouser.co.uk/ProductDetail/Weidmuller/1824420000?qs=BTG2th8YmhRalByZSURrtg%3D%3D" (at 204.47 680.01 0)
+    (property "Mouser Price/Stock" "1,11 €" (at 204.47 680.01 0)
       (effects (font (size 1.27 1.27)) (justify left top) hide)
     )

Commit message: update
Parts:
- F2, F3: value 100mA Polyfuse -> PTS120630V012
- H1, H2, H3, H4, H5, JP1: now left out of the parts list
- J3: value Phoenix_1776508 -> 1776508; PARTREV 06.02.2024 -> (none)
- J7: value Conn_01x02_Pin -> B2B-XH-AM(LF)(SN)
- R27: Manufacturer_Name (none) -> YAGEO; Manufacturer_Part_Number (none) -> RC0603FR-071KL; Mouser Part Number (none) -> 603-RC0603FR-071KL; Mouser Price/Stock (none) -> 0,009 €
Changed lines of the file:
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@@
       (effects (font (size 1.27 1.27)) (justify right))
     )
-    (property "Value" "100mA Polyfuse" (at 227.33 130.81 90)
+    (property "Value" "PTS120630V012" (at 227.33 130.81 90)
       (effects (font (size 1.27 1.27)) (justify right))
     )
@@
     )
     (property "Mouser Price/Stock" "0,108€" (at 219.71 128.27 0)
+      (effects (font (size 1.27 1.27)) hide)
+    )
+    (property "JLCPCB Part #" "" (at 219.71 128.27 0)
+      (effects (font (size 1.27 1.27)) hide)
+    )
+    (property "JLCPCB Price" "" (at 219.71 128.27 0)
       (effects (font (size 1.27 1.27)) hide)
     )
@@
     )
     (property "Mouser Price/Stock" "1,29 €" (at 242.57 143.51 0)
+      (effects (font (size 1.27 1.27)) hide)
+    )
+    (property "JLCPCB Part #" "" (at 242.57 143.51 0)
+      (effects (font (size 1.27 1.27)) hide)
+    )
+    (property "JLCPCB Price" "" (at 242.57 143.51 0)
       (effects (font (size 1.27 1.27)) hide)
     )
@@
   )
   (symbol (lib_id "Jumper:SolderJumper_3_Bridged12") (at 224.79 143.51 90) (mirror x) (unit 1)
-    (in_bom yes) (on_board yes) (dnp no) (fields_autoplaced)
+    (in_bom no) (on_board yes) (dnp no) (fields_autoplaced)
     (property "Reference" "JP1" (at 222.25 142.24 90)
       (effects (font (size 1.27 1.27)) (justify left))
@@
     )
     (property "Alternative Price" "" (at 224.79 143.51 0)
+      (effects (font (size 1.27 1.27)) hide)
+    )
+    (property "JLCPCB Part #" "" (at 224.79 143.51 0)
+      (effects (font (size 1.27 1.27)) hide)
+    )
+    (property "JLCPCB Price" "" (at 224.79 143.51 0)
       (effects (font (size 1.27 1.27)) hide)
     )
@@
       (effects (font (size 1.27 1.27)) (justify right))
     )
-    (property "Value" "Phoenix_1776508" (at 162.56 43.815 90)
+    (property "Value" "1776508" (at 162.56 43.815 90)
       (effects (font (size 1.27 1.27)) (justify right))
     )
@@
       (effects (font (size 1.27 1.27)) hide)
     )
-    (property "PARTREV" "06.02.2024" (at 161.29 43.18 0)
+    (property "PARTREV" "" (at 161.29 43.18 0)
       (effects (font (size 1.27 1.27)) (justify bottom) hide)
     )
@@
     )
     (property "Mouser Price/Stock" "1,83 €" (at 156.21 43.18 0)
+      (effects (font (size 1.27 1.27)) hide)
+    )
+    (property "JLCPCB Part #" "" (at 156.21 43.18 0)
+      (effects (font (size 1.27 1.27)) hide)
+    )
+    (property "JLCPCB Price" "" (at 156.21 43.18 0)
       (effects (font (size 1.27 1.27)) hide)
     )
@@
       (effects (font (size 1.27 1.27)) (justify right))
     )
-    (property "Value" "100mA Polyfuse" (at 242.57 146.05 90)
+    (property "Value" "PTS120630V012" (at 242.57 146.05 90)
       (effects (font (size 1.27 1.27)) (justify right))
     )
@@
       (effects (font (size 1.27 1.27)) hide)
     )
+    (property "JLCPCB Part #" "" (at 234.95 143.51 0)
+      (effects (font (size 1.27 1.27)) hide)
+    )
+    (property "JLCPCB Price" "" (at 234.95 143.51 0)
+      (effects (font (size 1.27 1.27)) hide)
+    )
     (pin "1")
     (pin "2")
@@
   )
   (symbol (lib_id "Mechanical:MountingHole") (at 114.3 144.78 0) (unit 1)
-    (in_bom yes) (on_board yes) (dnp no) (fields_autoplaced)
+    (in_bom no) (on_board yes) (dnp no) (fields_autoplaced)
     (property "Reference" "H3" (at 116.84 143.51 0)
       (effects (font (size 1.27 1.27)) (justify left))
@@
     )
     (property "Alternative Price" "" (at 114.3 144.78 0)
+      (effects (font (size 1.27 1.27)) hide)
+    )
+    (property "JLCPCB Part #" "" (at 114.3 144.78 0)
+      (effects (font (size 1.27 1.27)) hide)
+    )
+    (property "JLCPCB Price" "" (at 114.3 144.78 0)
       (effects (font (size 1.27 1.27)) hide)
     )
@@
       (effects (font (size 1.27 1.27)) (justify right))
     )
-    (property "Value" "Conn_01x02_Pin" (at 252.73 102.87 0)
+    (property "Value" "B2B-XH-AM(LF)(SN)" (at 252.73 102.87 0)
       (effects (font (size 1.27 1.27)) (justify right))
     )
@@
     )
     (property "Mouser Price/Stock" "0,152 €" (at 251.46 102.87 0)
+      (effects (font (size 1.27 1.27)) hide)
+    )
+    (property "Description" "B2B-XH-AM JST" (at 251.46 102.87 0)
+      (effects (font (size 1.27 1.27)) hide)
+    )
+    (property "JLCPCB Part #" "" (at 251.46 102.87 0)
+      (effects (font (size 1.27 1.27)) hide)
+    )
+    (property "JLCPCB Price" "" (at 251.46 102.87 0)
       (effects (font (size 1.27 1.27)) hide)
     )
@@
   )
   (symbol (lib_id "Mechanical:MountingHole") (at 48.26 144.78 0) (unit 1)
-    (in_bom yes) (on_board yes) (dnp no) (fields_autoplaced)
+    (in_bom no) (on_board yes) (dnp no) (fields_autoplaced)
     (property "Reference" "H1" (at 50.8 143.51 0)
       (effects (font (size 1.27 1.27)) (justify left))
@@
     )
     (property "Alternative Price" "" (at 48.26 144.78 0)
+      (effects (font (size 1.27 1.27)) hide)
+    )
+    (property "JLCPCB Part #" "" (at 48.26 144.78 0)
+      (effects (font (size 1.27 1.27)) hide)
+    )
+    (property "JLCPCB Price" "" (at 48.26 144.78 0)
       (effects (font (size 1.27 1.27)) hide)
     )
@@
       (effects (font (size 1.27 1.27)) hide)
     )
+    (property "JLCPCB Part #" "" (at 110.49 171.45 0)
+      (effects (font (size 1.27 1.27)) hide)
+    )
+    (property "JLCPCB Price" "" (at 110.49 171.45 0)
+      (effects (font (size 1.27 1.27)) hide)
+    )
     (pin "2")
     (pin "1")
@@
   )
   (symbol (lib_id "Mechanical:MountingHole_Pad") (at 114.3 163.83 0) (unit 1)
-    (in_bom yes) (on_board yes) (dnp no) (fields_autoplaced)
+    (in_bom no) (on_board yes) (dnp no) (fields_autoplaced)
     (property "Reference" "H5" (at 116.84 161.29 0)
       (effects (font (size 1.27 1.27)) (justify left))
@@
     )
     (property "Alternative Price" "" (at 114.3 163.83 0)
+      (effects (font (size 1.27 1.27)) hide)
+    )
+    (property "JLCPCB Part #" "" (at 114.3 163.83 0)
+      (effects (font (size 1.27 1.27)) hide)
+    )
+    (property "JLCPCB Price" "" (at 114.3 163.83 0)
       (effects (font (size 1.27 1.27)) hide)
     )
@@
   )
   (symbol (lib_id "Mechanical:MountingHole") (at 82.55 144.78 0) (unit 1)
-    (in_bom yes) (on_board yes) (dnp no) (fields_autoplaced)
+    (in_bom no) (on_board yes) (dnp no) (fields_autoplaced)
     (property "Reference" "H2" (at 85.09 143.51 0)
       (effects (font (size 1.27 1.27)) (justify left))
@@
       (effects (font (size 1.27 1.27)) hide)
     )
+    (property "JLCPCB Part #" "" (at 82.55 144.78 0)
+      (effects (font (size 1.27 1.27)) hide)
+    )
+    (property "JLCPCB Price" "" (at 82.55 144.78 0)
+      (effects (font (size 1.27 1.27)) hide)
+    )
     (instances
       (project "BugWiperPCB"
@@
     )
     (property "Alternative Price" "" (at 114.3 171.45 0)
+      (effects (font (size 1.27 1.27)) hide)
+    )
+    (property "Description" "SMD 1 kOhms 100mW 0603 1%" (at 114.3 171.45 0)
+      (effects (font (size 1.27 1.27)) hide)
+    )
+    (property "Manufacturer_Name" "YAGEO" (at 114.3 171.45 0)
+      (effects (font (size 1.27 1.27)) hide)
+    )
+    (property "Manufacturer_Part_Number" "RC0603FR-071KL" (at 114.3 171.45 0)
+      (effects (font (size 1.27 1.27)) hide)
+    )
+    (property "Mouser Part Number" "603-RC0603FR-071KL" (at 114.3 171.45 0)
+      (effects (font (size 1.27 1.27)) hide)
+    )
+    (property "Mouser Price/Stock" "0,009 €" (at 114.3 171.45 0)
+      (effects (font (size 1.27 1.27)) hide)
+    )
+    (property "JLCPCB Part #" "" (at 114.3 171.45 0)
+      (effects (font (size 1.27 1.27)) hide)
+    )
+    (property "JLCPCB Price" "" (at 114.3 171.45 0)
       (effects (font (size 1.27 1.27)) hide)
     )
@@
       (effects (font (size 1.27 1.27)) hide)
     )
+    (property "JLCPCB Part #" "" (at 187.96 85.09 0)
+      (effects (font (size 1.27 1.27)) hide)
+    )
+    (property "JLCPCB Price" "" (at 187.96 85.09 0)
+      (effects (font (size 1.27 1.27)) hide)
+    )
     (pin "3")
     (pin "4")
@@
   )
   (symbol (lib_id "Mechanical:MountingHole") (at 48.26 162.56 0) (unit 1)
-    (in_bom yes) (on_board yes) (dnp no) (fields_autoplaced)
+    (in_bom no) (on_board yes) (dnp no) (fields_autoplaced)
     (property "Reference" "H4" (at 50.8 161.29 0)
       (effects (font (size 1.27 1.27)) (justify left))
@@
       (effects (font (size 1.27 1.27)) hide)
     )
+    (property "JLCPCB Part #" "" (at 48.26 162.56 0)
+      (effects (font (size 1.27 1.27)) hide)
+    )
+    (property "JLCPCB Price" "" (at 48.26 162.56 0)
+      (effects (font (size 1.27 1.27)) hide)
+    )

Commit message: update BOM
Parts:
- added J9: 1873207, symbol Connector:Conn_01x02_Socket
- F2, F3: Price 0,108€ -> (none)
- J3: MANUFACTURER Phoenix Contact -> (none)
- J6: Height 8.5 -> (none)
- J7: now not fitted; now left out of the parts list
Changed lines of the file:
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@@
-      (effects (font (size 1.27 1.27)) hide)
-    )
-    (property "Price" "0,108€" (at 219.71 128.27 0)
       (effects (font (size 1.27 1.27)) hide)
     )
@@
       (effects (font (size 1.27 1.27)) hide)
     )
-    (property "PARTREV" "" (at 161.29 43.18 0)
-      (effects (font (size 1.27 1.27)) (justify bottom) hide)
-    )
-    (property "STANDARD" "" (at 151.13 43.18 0)
-      (effects (font (size 1.27 1.27)) (justify bottom) hide)
-    )
     (property "MAXIMUM_PACKAGE_HEIGHT" "8.75mm" (at 156.21 43.18 0)
       (effects (font (size 1.27 1.27)) (justify bottom) hide)
     )
-    (property "MANUFACTURER" "Phoenix Contact" (at 153.67 43.18 0)
-      (effects (font (size 1.27 1.27)) (justify bottom) hide)
-    )
     (property "Manufacturer_Name" "Phoenix Contact" (at 156.21 43.18 0)
       (effects (font (size 1.27 1.27)) hide)
@@
         (path "/d31a15bd-db02-4d4c-9593-17c596d3182c"
           (reference "J3") (unit 1)
+        )
+      )
+    )
+  )
+  (symbol (lib_id "Connector:Conn_01x02_Socket") (at 156.21 34.29 90) (mirror x) (unit 1)
+    (in_bom yes) (on_board no) (dnp no)
+    (property "Reference" "J9" (at 154.94 32.385 90)
+      (effects (font (size 1.27 1.27)) (justify left))
+    )
+    (property "Value" "1873207" (at 154.94 34.925 90)
+      (effects (font (size 1.27 1.27)) (justify left))
+    )
+    (property "Footprint" "" (at 156.21 34.29 0)
+      (effects (font (size 1.27 1.27)) hide)
+    )
+    (property "Datasheet" "~" (at 156.21 34.29 0)
+      (effects (font (size 1.27 1.27)) hide)
+    )
+    (property "Manufacturer_Name" "Phoenix Contact" (at 156.21 34.29 0)
+      (effects (font (size 1.27 1.27)) hide)
+    )
+    (property "Manufacturer_Part_Number" "1873207" (at 156.21 34.29 0)
+      (effects (font (size 1.27 1.27)) hide)
+    )
+    (property "Mouser Part Number" "651-1873207" (at 156.21 34.29 0)
+      (effects (font (size 1.27 1.27)) hide)
+    )
+    (property "Mouser Price/Stock" "2,51€" (at 156.21 34.29 0)
+      (effects (font (size 1.27 1.27)) hide)
+    )
+    (pin "2")
+    (pin "1")
+    (instances
+      (project "BugWiperPCB"
+        (path "/d31a15bd-db02-4d4c-9593-17c596d3182c"
+          (reference "J9") (unit 1)
         )
       )
@@
       (effects (font (size 1.27 1.27)) hide)
     )
-    (property "Price" "0,108€" (at 234.95 143.51 0)
-      (effects (font (size 1.27 1.27)) hide)
-    )
     (property "Alternative MF" "" (at 234.95 143.51 0)
       (effects (font (size 1.27 1.27)) hide)
@@
   )
   (symbol (lib_id "Connector:Conn_01x02_Pin") (at 251.46 102.87 180) (unit 1)
-    (in_bom yes) (on_board yes) (dnp no) (fields_autoplaced)
+    (in_bom no) (on_board yes) (dnp yes) (fields_autoplaced)
     (property "Reference" "J7" (at 252.73 100.33 0)
       (effects (font (size 1.27 1.27)) (justify right))
@@
       (effects (font (size 1.27 1.27)) (justify left top) hide)
     )
-    (property "Height" "8.5" (at 204.47 480.01 0)
-      (effects (font (size 1.27 1.27)) (justify left top) hide)
-    )

Commit message: update PCB to view Values and Refs
Parts:
- C27: value 100nF -> 100nF
Changed lines of the file:
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@@
       (effects (font (size 1.27 1.27)) (justify left))
     )
-    (property "Value" "100nF " (at 106.68 172.72 0)
+    (property "Value" "100nF" (at 106.68 172.72 0)
       (effects (font (size 1.27 1.27)) (justify left))
     )
