File: Hardware/ControllerPCB/BugWiperPCB.kicad_pcb (KiCad board)
At the start: 4 copper layers, 110 x 40 mm, 115 parts, among them J1 UJ20-C-H-G-SMT-1-P16-TR, J2 1770924, J3 1776508, J4 54602-908LF, J5 Conn_TagConnect_TC2030-NL_ESP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, J6 1824420000, J7 B2B-XH-AM(LF)(SN), J8 104031-0811, Q1 SQJ146ELP, SW1 SW_Push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

Commit message: fix schematics and pins for the encoder
Parts:
- C36: value 10nF -> 100nF
- C38: value 100nF -> 10nF
Connections:
- C36 pad 1: Enc1 -> SW2
- C37 pad 1: Enc2 -> Enc1
- C38 pad 1: SW1 -> Enc2
- C39 pad 1: SW2 -> SW1
- RN5 pad 5: SW2 -> SW1
- RN5 pad 6: SW1 -> Enc2
- RN5 pad 7: Enc2 -> Enc1
- RN5 pad 8: Enc1 -> SW2
- U1 pad 10: SW1 -> Enc2
- U1 pad 11: SW2 -> SW1
- U1 pad 8: Enc1 -> SW2
- U1 pad 9: Enc2 -> Enc1
Routing:
- net Enc1: track 8.82 -> 4.86 mm, vias 2 -> 0
- net SW1: track 4.12 -> 6.66 mm
- net SW2: track 6.66 -> 8.82 mm, vias 0 -> 2
- net Enc2: track 4.86 -> 4.12 mm

Commit message: update controller PCB: change Encoder filter to 1nF add 0 Ohm resistor for JP1 to BOM
Parts:
- C37, C38: value 10nF -> 1nF
Changed lines of the file:
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@@
         (effects (font (size 1 1) (thickness 0.15)))
     )
-    (fp_text value "10nF" (at 0 0 -90) (layer "User.6")
+    (fp_text value "1nF" (at 0 0 -90) (layer "User.6")
         (effects (font (size 0.6 0.6) (thickness 0.08)))
     )
@@
         (effects (font (size 1 1) (thickness 0.15)))
     )
-    (fp_text value "10nF" (at 0 0 90) (layer "User.6")
+    (fp_text value "1nF" (at 0 0 90) (layer "User.6")
         (effects (font (size 0.6 0.6) (thickness 0.08)))
     )

Commit message: Update PCB files and documentation for BugWiper 2.0: change revision to V1.2, update value from C4 from 100nF to 470nF
Parts:
- C4: value 100nF -> 470nF
- JP1: value SolderJumper_3_Open -> SolderJumper_0R_0603
Changed lines of the file:
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@@
   (title_block
     (title "BugWiper2.0 Controller PCB")
-    (date "2025-05-10")
-    (rev "1.0")
+    (date "2026-05-04")
+    (rev "1.2")
   )
   (layers
@@
     (property "Alternative PN" "")
     (property "Alternative Price" "")
-    (property "Description" "100nF+/-10% 50V X7R 0603")
+    (property "Description" "470nF+/-10% 25V X7R 0603")
     (property "JLCPCB Part #" "")
     (property "JLCPCB Price" "")
     (property "Manufacturer_Name" "Samsung")
-    (property "Manufacturer_Part_Number" "CL10B104KB8NNNC")
-    (property "Mouser Part Number" "187-CL10B104KB8NNNC")
+    (property "Manufacturer_Part_Number" "CL10B474KA8NFNC")
+    (property "Mouser Part Number" "187-CL10B474KA8NFNC")
     (property "Mouser Price/Stock" "0,01 €")
     (property "Sheetfile" "ESP32-S3.kicad_sch")
@@
         (effects (font (size 1 1) (thickness 0.15)))
     )
-    (fp_text value "100nF" (at 0 0 180) (layer "User.6")
+    (fp_text value "470nF" (at 0 0 180) (layer "User.6")
         (effects (font (size 0.6 0.6) (thickness 0.08)))
     )
@@
     (property "Alternative PN" "")
     (property "Alternative Price" "")
+    (property "Description" "SMD 0 Ohms 100mW 0603 1%")
     (property "JLCPCB Part #" "")
     (property "JLCPCB Price" "")
+    (property "Manufacturer_Name" "YAGEO")
+    (property "Manufacturer_Part_Number" "RC0603FR-070RL")
+    (property "Mouser Part Number" "603-RC0603FR-070RL")
+    (property "Mouser Price/Stock" "0,095€")
     (property "Sheetfile" "BugWiperPCB.kicad_sch")
     (property "Sheetname" "")
@@
         (effects (font (size 1 1) (thickness 0.15)))
     )
-    (fp_text value "SolderJumper_3_Open" (at 0 1.9 90) (layer "F.Fab") hide
+    (fp_text value "SolderJumper_0R_0603" (at 0 1.9 90) (layer "F.Fab") hide
         (effects (font (size 1 1) (thickness 0.15)))
     )
