File: Hardware/ControllerPCB/ESP32-S3.kicad_sch (KiCad schematic)
At the start: 55 parts, among them J1 UJ20-C-H-G-SMT-1-P16-TR, J4 54602-908LF, J5 Conn_TagConnect_TC2030-NL_ESP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, J8 104031-0811, SW1 SW_Push, SW2 SW_Push, U1 ESP32-S3-WROOM-1, U7 AP7333-33SRG-7

Commit message: update BOM
Parts:
- C40: Manufacturer_Name (none) -> Samsung; Manufacturer_Part_Number (none) -> CL21B105MBFNNNE; Mouser Part Number (none) -> 187-CL21B105MBFNNNE; Mouser Price/Stock (none) -> 0,026€
- CR1, CR2, CR3, CR4: Price 0,233 -> (none)
- D1: Price 0,21 -> (none)
- F1, F4: MP PTS120630V012 -> (none); Price 0,108€ -> (none)
- J1: Availability In Stock -> (none); Check_prices https://www.snapeda.com/parts/UJ20-C-H-G-SMT-1-P16-TR/Same+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 -> (none); MANUFACTURER Same Sky -> (none); MF Same Sky -> (none); MP UJ20-C-H-G-SMT-1-P16-TR -> (none); Price None -> (none)
- JP2, JP3, R16, R17: now left out of the parts list
- RN1, RN2, RN5: Price 0,04€ -> (none)
- RN3, RN4, RN6, RN7, RN8: Price 0,10€ -> (none)
Changed lines of the file:
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@@
   )
   (symbol (lib_id "Device:R") (at 29.21 107.95 180) (unit 1)
-    (in_bom yes) (on_board yes) (dnp yes)
+    (in_bom no) (on_board yes) (dnp yes)
     (property "Reference" "R16" (at 26.67 107.95 90)
       (effects (font (size 1.27 1.27)))
@@
       (effects (font (size 1.27 1.27)) hide)
     )
-    (property "Price" "0,10€" (at 55.88 173.99 0)
-      (effects (font (size 1.27 1.27)) hide)
-    )
     (property "Mouser Price/Stock" " 0,085 € " (at 55.88 173.99 0)
       (effects (font (size 1.27 1.27)) hide)
@@
       (effects (font (size 1.27 1.27)) hide)
     )
-    (property "Price" "0,04€" (at 266.7 106.68 0)
-      (effects (font (size 1.27 1.27)) hide)
-    )
     (property "Mouser Price/Stock" " 0,034 € " (at 266.7 106.68 0)
       (effects (font (size 1.27 1.27)) hide)
@@
       (effects (font (size 1.27 1.27)) hide)
     )
-    (property "MP" "PTS120630V012" (at 17.78 146.05 0)
-      (effects (font (size 1.27 1.27)) hide)
-    )
     (property "Manufacturer_Name" "Eaton Electronics" (at 17.78 146.05 0)
       (effects (font (size 1.27 1.27)) hide)
@@
       (effects (font (size 1.27 1.27)) hide)
     )
-    (property "Price" "0,108€" (at 17.78 146.05 0)
-      (effects (font (size 1.27 1.27)) hide)
-    )
     (property "Alternative MF" "" (at 17.78 146.05 0)
       (effects (font (size 1.27 1.27)) hide)
@@
   )
   (symbol (lib_id "BugWiper_Lib:SolderJumper_2_Bridged") (at 29.21 97.79 90) (mirror x) (unit 1)
-    (in_bom yes) (on_board yes) (dnp no) (fields_autoplaced)
+    (in_bom no) (on_board yes) (dnp no) (fields_autoplaced)
     (property "Reference" "JP3" (at 31.75 96.52 90)
       (effects (font (size 1.27 1.27)) (justify right))
@@
       (effects (font (size 1.27 1.27)) hide)
     )
-    (property "Price" "0,10€" (at 204.47 148.59 0)
-      (effects (font (size 1.27 1.27)) hide)
-    )
     (property "Mouser Price/Stock" " 0,098 € " (at 204.47 148.59 0)
       (effects (font (size 1.27 1.27)) hide)
@@
       (effects (font (size 1.27 1.27)) hide)
     )
-    (property "Price" "0,10€" (at 33.02 161.29 0)
-      (effects (font (size 1.27 1.27)) hide)
-    )
     (property "Mouser Price/Stock" " 0,098 € " (at 33.02 161.29 0)
       (effects (font (size 1.27 1.27)) hide)
@@
       (effects (font (size 1.27 1.27)) hide)
     )
-    (property "MP" "PTS120630V012" (at 49.53 138.43 0)
-      (effects (font (size 1.27 1.27)) hide)
-    )
     (property "Manufacturer_Name" "Eaton Electronics" (at 49.53 138.43 0)
       (effects (font (size 1.27 1.27)) hide)
@@
       (effects (font (size 1.27 1.27)) hide)
     )
-    (property "Price" "0,108€" (at 49.53 138.43 0)
-      (effects (font (size 1.27 1.27)) hide)
-    )
     (property "Alternative MF" "" (at 49.53 138.43 0)
       (effects (font (size 1.27 1.27)) hide)
@@
       (effects (font (size 1.27 1.27)) hide)
     )
-    (property "Price" "0,10€" (at 204.47 143.51 0)
-      (effects (font (size 1.27 1.27)) hide)
-    )
     (property "Mouser Price/Stock" " 0,098 € " (at 204.47 143.51 0)
       (effects (font (size 1.27 1.27)) hide)
@@
       (effects (font (size 1.27 1.27)) hide)
     )
-    (property "MF" "Same Sky" (at 21.59 41.91 0)
-      (effects (font (size 1.27 1.27)) (justify bottom) hide)
-    )
     (property "MAXIMUM_PACKAGE_HEIGHT" "3.46mm" (at 21.59 41.91 0)
       (effects (font (size 1.27 1.27)) (justify bottom) hide)
@@
       (effects (font (size 1.27 1.27)) (justify bottom) hide)
     )
-    (property "Price" "None" (at 21.59 41.91 0)
-      (effects (font (size 1.27 1.27)) (justify bottom) hide)
-    )
-    (property "Check_prices" "https://www.snapeda.com/parts/UJ20-C-H-G-SMT-1-P16-TR/Same+Sky/view-part/?ref=eda" (at 21.59 41.91 0)
-      (effects (font (size 1.27 1.27)) (justify bottom) hide)
-    )
-    (property "STANDARD" "" (at 21.59 41.91 0)
-      (effects (font (size 1.27 1.27)) (justify bottom) hide)
-    )
-    (property "PARTREV" "" (at 21.59 41.91 0)
-      (effects (font (size 1.27 1.27)) (justify bottom) hide)
-    )
-    (property "SnapEDA_Link" "" (at 21.59 41.91 0)
-      (effects (font (size 1.27 1.27)) (justify bottom) hide)
-    )
-    (property "MP" "UJ20-C-H-G-SMT-1-P16-TR" (at 21.59 41.91 0)
-      (effects (font (size 1.27 1.27)) (justify bottom) hide)
-    )
     (property "Description" "\n                        \n                            USB-C (USB TYPE-C) USB 2.0 Receptacle Connector 24 (16+8 Dummy) Position Surface Mount, Right Angle; Through Hole\n                        \n" (at 21.59 41.91 0)
       (effects (font (size 1.27 1.27)) (justify bottom) hide)
     )
-    (property "Availability" "In Stock" (at 21.59 41.91 0)
-      (effects (font (size 1.27 1.27)) (justify bottom) hide)
-    )
-    (property "MANUFACTURER" "Same Sky" (at 21.59 41.91 0)
-      (effects (font (size 1.27 1.27)) (justify bottom) hide)
-    )
     (property "Manufacturer_Name" "Same Sky" (at 21.59 41.91 0)
       (effects (font (size 1.27 1.27)) hide)
@@
       (effects (font (size 1.27 1.27)) hide)
     )
-    (property "Price" "0,04€" (at 266.7 127 0)
-      (effects (font (size 1.27 1.27)) hide)
-    )
     (property "Mouser Price/Stock" " 0,034 € " (at 266.7 127 0)
       (effects (font (size 1.27 1.27)) hide)
@@
       (effects (font (size 1.27 1.27)) hide)
     )
-    (property "Price" "0,233" (at 180.34 25.4 0)
-      (effects (font (size 1.27 1.27)) hide)
-    )
     (property "Mouser Price/Stock" "0,233€" (at 180.34 25.4 0)
       (effects (font (size 1.27 1.27)) hide)
@@
   )
   (symbol (lib_id "Device:R") (at 57.15 107.95 180) (unit 1)
-    (in_bom yes) (on_board yes) (dnp yes)
+    (in_bom no) (on_board yes) (dnp yes)
     (property "Reference" "R17" (at 54.61 107.95 90)
       (effects (font (size 1.27 1.27)))
@@
       (effects (font (size 1.27 1.27)) hide)
     )
-    (property "Price" "0,10€" (at 153.67 160.02 0)
-      (effects (font (size 1.27 1.27)) hide)
-    )
     (property "Mouser Price/Stock" " 0,085 € " (at 153.67 160.02 0)
       (effects (font (size 1.27 1.27)) hide)
@@
   )
   (symbol (lib_id "BugWiper_Lib:SolderJumper_2_Bridged") (at 57.15 97.79 90) (mirror x) (unit 1)
-    (in_bom yes) (on_board yes) (dnp no)
+    (in_bom no) (on_board yes) (dnp no)
     (property "Reference" "JP2" (at 53.34 96.52 90)
       (effects (font (size 1.27 1.27)))
@@
       (effects (font (size 1.27 1.27)) hide)
     )
+    (property "Description" "1uF 50V X7R 0805" (at 140.97 40.64 0)
+      (effects (font (size 1.27 1.27)) hide)
+    )
+    (property "Manufacturer_Name" "Samsung" (at 140.97 40.64 0)
+      (effects (font (size 1.27 1.27)) hide)
+    )
+    (property "Manufacturer_Part_Number" "CL21B105MBFNNNE" (at 140.97 40.64 0)
+      (effects (font (size 1.27 1.27)) hide)
+    )
+    (property "Mouser Part Number" "187-CL21B105MBFNNNE" (at 140.97 40.64 0)
+      (effects (font (size 1.27 1.27)) hide)
+    )
+    (property "Mouser Price/Stock" "0,026€" (at 140.97 40.64 0)
+      (effects (font (size 1.27 1.27)) hide)
+    )
     (pin "1")
     (pin "2")
@@
       (effects (font (size 1.27 1.27)) hide)
     )
-    (property "Price" "0,233" (at 35.56 34.29 0)
-      (effects (font (size 1.27 1.27)) hide)
-    )
     (property "Mouser Price/Stock" "0,233€" (at 35.56 34.29 0)
       (effects (font (size 1.27 1.27)) hide)
@@
       (effects (font (size 1.27 1.27)) hide)
     )
-    (property "Price" "0,21" (at 40.64 21.59 0)
-      (effects (font (size 1.27 1.27)) hide)
-    )
     (property "Mouser Price/Stock" "0,209€" (at 40.64 21.59 0)
       (effects (font (size 1.27 1.27)) hide)
@@
       (effects (font (size 1.27 1.27)) hide)
     )
-    (property "Price" "0,10€" (at 53.34 152.4 0)
-      (effects (font (size 1.27 1.27)) hide)
-    )
     (property "Mouser Price/Stock" " 0,098 € " (at 53.34 152.4 0)
       (effects (font (size 1.27 1.27)) hide)
@@
       (effects (font (size 1.27 1.27)) hide)
     )
-    (property "Price" "0,10€" (at 204.47 146.05 0)
-      (effects (font (size 1.27 1.27)) hide)
-    )
     (property "Mouser Price/Stock" " 0,098 € " (at 204.47 146.05 0)
       (effects (font (size 1.27 1.27)) hide)
@@
       (effects (font (size 1.27 1.27)) hide)
     )
-    (property "Price" "0,10€" (at 25.4 144.78 0)
-      (effects (font (size 1.27 1.27)) hide)
-    )
     (property "Mouser Price/Stock" " 0,098 € " (at 25.4 144.78 0)
       (effects (font (size 1.27 1.27)) hide)
@@
       (effects (font (size 1.27 1.27)) hide)
     )
-    (property "Price" "0,10€" (at 22.86 144.78 0)
-      (effects (font (size 1.27 1.27)) hide)
-    )
     (property "Mouser Price/Stock" " 0,098 € " (at 22.86 144.78 0)
       (effects (font (size 1.27 1.27)) hide)
@@
       (effects (font (size 1.27 1.27)) hide)
     )
-    (property "Price" "0,233" (at 57.15 186.69 0)
-      (effects (font (size 1.27 1.27)) hide)
-    )
     (property "Mouser Price/Stock" "0,233€" (at 57.15 186.69 0)
       (effects (font (size 1.27 1.27)) hide)
@@
       (effects (font (size 1.27 1.27)) hide)
     )
-    (property "Price" "0,233" (at 204.47 153.67 0)
-      (effects (font (size 1.27 1.27)) hide)
-    )
     (property "Mouser Price/Stock" "0,233€" (at 204.47 153.67 0)
       (effects (font (size 1.27 1.27)) hide)
@@
       (effects (font (size 1.27 1.27)) hide)
     )
-    (property "Price" "0,10€" (at 204.47 140.97 0)
-      (effects (font (size 1.27 1.27)) hide)
-    )
     (property "Mouser Price/Stock" " 0,098 € " (at 204.47 140.97 0)
       (effects (font (size 1.27 1.27)) hide)
@@
       (effects (font (size 1.27 1.27)) hide)
     )
-    (property "Price" "0,04€" (at 247.65 146.05 0)
-      (effects (font (size 1.27 1.27)) hide)
-    )
     (property "Mouser Price/Stock" " 0,034 € " (at 247.65 146.05 0)
       (effects (font (size 1.27 1.27)) hide)
@@
       (effects (font (size 1.27 1.27)) hide)
     )
-    (property "Price" "0,10€" (at 53.34 154.94 0)
-      (effects (font (size 1.27 1.27)) hide)
-    )

Commit message: update PCB to view Values and Refs
Parts:
- C22, C29, C3, C30, C38, C39: value 100nF -> 100nF
- C32, C33, C34, C35, C36, C37: value 10nF -> 10nF
- C4: value 100nF -> 100nF; footprint Capacitor_SMD:C_0603_1608Metric -> BugWiper_lib:C_0603_1608Metric
- C40: value 1uF 50V -> 1uF
- RN1, RN2, RN5: value 1k x 4 -> 4x1k
- RN3, RN6, RN7: value 100R x 4 -> 4x100R
- RN4, RN8: value 10k x 4 -> 4x10k
Changed lines of the file:
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@@
       (effects (font (size 1.27 1.27)))
     )
-    (property "Value" "10k x 4" (at 55.88 166.37 90)
+    (property "Value" "4x10k" (at 55.88 166.37 90)
       (effects (font (size 1.27 1.27)))
     )
@@
       (effects (font (size 1.27 1.27)) (justify left))
     )
-    (property "Value" "10nF " (at 248.92 158.75 0)
+    (property "Value" "10nF" (at 248.92 158.75 0)
       (effects (font (size 1.27 1.27)) (justify left))
     )
@@
       (effects (font (size 1.27 1.27)))
     )
-    (property "Value" "1k x 4" (at 266.7 100.33 90)
+    (property "Value" "4x1k" (at 266.7 100.33 90)
       (effects (font (size 1.27 1.27)))
     )
@@
       (effects (font (size 1.27 1.27)) (justify left))
     )
-    (property "Value" "10nF " (at 62.23 185.42 0)
+    (property "Value" "10nF" (at 62.23 185.42 0)
       (effects (font (size 1.27 1.27)) (justify left))
     )
@@
       (effects (font (size 1.27 1.27)) (justify left))
     )
-    (property "Value" "100R x 4" (at 198.12 143.51 90)
+    (property "Value" "4x100R" (at 198.12 143.51 90)
       (effects (font (size 1.27 1.27)) (justify left) hide)
     )
@@
       (effects (font (size 1.27 1.27)))
     )
-    (property "Value" "100R x 4" (at 40.64 161.29 90)
+    (property "Value" "4x100R" (at 40.64 161.29 90)
       (effects (font (size 1.27 1.27)))
     )
@@
       (effects (font (size 1.27 1.27)) (justify left))
     )
-    (property "Value" "100nF " (at 231.14 38.1 0)
+    (property "Value" "100nF" (at 231.14 38.1 0)
       (effects (font (size 1.27 1.27)) (justify left))
     )
@@
       (effects (font (size 1.27 1.27)) (justify left))
     )
-    (property "Value" "100R x 4" (at 198.12 138.43 90)
+    (property "Value" "4x100R" (at 198.12 138.43 90)
       (effects (font (size 1.27 1.27)) (justify left) hide)
     )
@@
       (effects (font (size 1.27 1.27)))
     )
-    (property "Value" "1k x 4" (at 266.7 118.11 90)
+    (property "Value" "4x1k" (at 266.7 118.11 90)
       (effects (font (size 1.27 1.27)))
     )
@@
       (effects (font (size 1.27 1.27)) (justify left))
     )
-    (property "Value" "10k x 4" (at 146.05 154.94 90)
+    (property "Value" "4x10k" (at 146.05 154.94 90)
       (effects (font (size 1.27 1.27)) (justify left))
     )
@@
       (effects (font (size 1.27 1.27)) (justify left))
     )
-    (property "Value" "100nF " (at 86.36 27.94 0)
+    (property "Value" "100nF" (at 86.36 27.94 0)
       (effects (font (size 1.27 1.27)) (justify left))
     )
@@
       (effects (font (size 1.27 1.27)) (justify left))
     )
-    (property "Value" "1uF 50V" (at 142.24 44.45 90)
+    (property "Value" "1uF" (at 142.24 44.45 90)
       (effects (font (size 1.27 1.27)) (justify left))
     )
@@
       (effects (font (size 1.27 1.27)) (justify left))
     )
-    (property "Value" "100nF " (at 260.35 38.1 0)
+    (property "Value" "100nF" (at 260.35 38.1 0)
       (effects (font (size 1.27 1.27)) (justify left))
     )
-    (property "Footprint" "Capacitor_SMD:C_0603_1608Metric" (at 265.1252 39.37 0)
+    (property "Footprint" "BugWiper_lib:C_0603_1608Metric" (at 265.1252 39.37 0)
       (effects (font (size 1.27 1.27)) hide)
     )
@@
       (effects (font (size 1.27 1.27)) (justify left))
     )
-    (property "Value" "10nF " (at 57.15 185.42 0)
+    (property "Value" "10nF" (at 57.15 185.42 0)
       (effects (font (size 1.27 1.27)) (justify left))
     )
@@
       (effects (font (size 1.27 1.27)) (justify left))
     )
-    (property "Value" "10nF " (at 255.27 158.75 0)
+    (property "Value" "10nF" (at 255.27 158.75 0)
       (effects (font (size 1.27 1.27)) (justify left))
     )
@@
       (effects (font (size 1.27 1.27)) (justify left))
     )
-    (property "Value" "100nF " (at 147.32 22.86 0)
+    (property "Value" "100nF" (at 147.32 22.86 0)
       (effects (font (size 1.27 1.27)) (justify left))
     )
@@
       (effects (font (size 1.27 1.27)) (justify left))
     )
-    (property "Value" "100nF " (at 261.62 158.75 0)
+    (property "Value" "100nF" (at 261.62 158.75 0)
       (effects (font (size 1.27 1.27)) (justify left))
     )
@@
       (effects (font (size 1.27 1.27)) (justify left))
     )
-    (property "Value" "100R x 4" (at 52.07 154.94 0)
+    (property "Value" "4x100R" (at 52.07 154.94 0)
       (effects (font (size 1.27 1.27)) (justify left) hide)
     )
@@
       (effects (font (size 1.27 1.27)) (justify left))
     )
-    (property "Value" "100R x 4" (at 198.12 140.97 90)
+    (property "Value" "4x100R" (at 198.12 140.97 90)
       (effects (font (size 1.27 1.27)) (justify left) hide)
     )
@@
       (effects (font (size 1.27 1.27)) (justify left))
     )
-    (property "Value" "10nF " (at 67.31 185.42 0)
+    (property "Value" "10nF" (at 67.31 185.42 0)
       (effects (font (size 1.27 1.27)) (justify left))
     )
@@
       (effects (font (size 1.27 1.27)) (justify left))
     )
-    (property "Value" "100R x 4" (at 20.32 138.43 90)
+    (property "Value" "4x100R" (at 20.32 138.43 90)
       (effects (font (size 1.27 1.27)) (justify left) hide)
     )
@@
       (effects (font (size 1.27 1.27)) (justify left))
     )
-    (property "Value" "100nF " (at 121.92 27.94 0)
+    (property "Value" "100nF" (at 121.92 27.94 0)
       (effects (font (size 1.27 1.27)) (justify left))
     )
@@
       (effects (font (size 1.27 1.27)) (justify left))
     )
-    (property "Value" "100nF " (at 267.97 158.75 0)
+    (property "Value" "100nF" (at 267.97 158.75 0)
       (effects (font (size 1.27 1.27)) (justify left))
     )
@@
       (effects (font (size 1.27 1.27)) (justify left))
     )
-    (property "Value" "10nF " (at 72.39 185.42 0)
+    (property "Value" "10nF" (at 72.39 185.42 0)
       (effects (font (size 1.27 1.27)) (justify left))
     )
@@
       (effects (font (size 1.27 1.27)) (justify left))
     )
-    (property "Value" "100R x 4" (at 17.78 138.43 90)
+    (property "Value" "4x100R" (at 17.78 138.43 90)
       (effects (font (size 1.27 1.27)) (justify left) hide)
     )
@@
       (effects (font (size 1.27 1.27)) (justify left))
     )
-    (property "Value" "100R x 4" (at 203.2 143.51 0)
+    (property "Value" "4x100R" (at 203.2 143.51 0)
       (effects (font (size 1.27 1.27)) (justify left) hide)
     )
@@
       (effects (font (size 1.27 1.27)))
     )
-    (property "Value" "1k x 4" (at 247.65 137.16 90)
+    (property "Value" "4x1k" (at 247.65 137.16 90)
       (effects (font (size 1.27 1.27)))
     )
@@
       (effects (font (size 1.27 1.27)) (justify left))
     )
-    (property "Value" "100R x 4" (at 46.99 149.86 90)
+    (property "Value" "4x100R" (at 46.99 149.86 90)
       (effects (font (size 1.27 1.27)) (justify left) hide)
     )

Commit message: update Controller PCB PDF Export and layer of Values and Reference
Parts:
- CR1, CR2, CR3, CR4: value D5V0P4UR6SO-7 -> D5V0P4UR6
Changed lines of the file:
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@@
       (effects (font (size 1.524 1.524)))
     )
-    (property "Value" "D5V0P4UR6SO-7" (at 201.93 34.29 0)
+    (property "Value" "D5V0P4UR6" (at 201.93 34.29 0)
       (effects (font (size 1.524 1.524)))
     )
@@
       (effects (font (size 1.524 1.524)))
     )
-    (property "Value" "D5V0P4UR6SO-7" (at 55.88 38.1 0)
+    (property "Value" "D5V0P4UR6" (at 55.88 38.1 0)
       (effects (font (size 1.524 1.524)))
     )
@@
       (effects (font (size 1.524 1.524)))
     )
-    (property "Value" "D5V0P4UR6SO-7" (at 36.83 190.5 0)
+    (property "Value" "D5V0P4UR6" (at 36.83 190.5 0)
       (effects (font (size 1.524 1.524)))
     )
@@
       (effects (font (size 1.524 1.524)))
     )
-    (property "Value" "D5V0P4UR6SO-7" (at 224.79 163.83 0)
+    (property "Value" "D5V0P4UR6" (at 224.79 163.83 0)
       (effects (font (size 1.524 1.524)))
     )
