File: Hardware/ControllerPCB/Power.kicad_sch (KiCad schematic)
At the start: 46 parts, among them Q1 SQJ146ELP, U2 BTN9960LV, U3 BTN9960LV, U4 INA180A2, U6 TSR 0.5-2433

Commit message: update controller PCB: change Encoder filter to 1nF add 0 Ohm resistor for JP1 to BOM
Other:
- company: (none) -> M. Scholjegerdes
- title: (none) -> BugWiper 2.0 Controller PCB
Changed lines of the file:
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@@
 (kicad_sch (version 20230121) (generator eeschema)
   (paper "A4")
+  (title_block
+    (title "BugWiper 2.0 Controller PCB")
+    (date "2025-06-02")
+    (rev "V1.1")
+    (company "M. Scholjegerdes")
+  )
   (junction (at 242.57 50.8) (diameter 0) (color 0 0 0 0)
   )
